File: korsotracker/korsotracker.sch (KiCad schematic (older format))
At the start: 14 parts

Commit message: Schematics op amp
Schematics drawing now with op amp to audio out
Parts:
- removed U?: OPA365, symbol OPA365
- added C?: tbd, ~, symbol CSMALL
- added C?: CSMALL, ~, symbol CSMALL
- added R? (x2): JUMPER, ~, symbol R
- added R?: tbd, ~, symbol R
- added RV?: POT, ~, symbol POT
- added U?: TLV271, symbol TLV271
- Q?: value MOSFET_P -> DMP1045U
- R?: renamed from tbd; value R -> tbd
Connections:
- net labels added: +3.3V, AUDIO OUT
- wire segments 31 -> 55
Changed lines of the file:
@@
-$EndComp
-$Comp
-L OPA365 U?
-U 1 1 55329966
-P 4000 6250
-F 0 "U?" H 4000 6250 60  0000 C CNN
-F 1 "OPA365" H 4000 5500 60  0000 C CNN
-F 2 "" H 4000 6250 60  0000 C CNN
-F 3 "" H 4000 6250 60  0000 C CNN
-	1    4000 6250
-	1    0    0    -1
 $EndComp
 $Comp
@@
 	8400 1900 8700 1900
 $Comp
-L R tbd
+L R R?
 U 1 1 5532A3B6
 P 9250 900
-F 0 "tbd" V 9330 900 40  0000 C CNN
-F 1 "R" V 9257 901 40  0000 C CNN
+F 0 "R?" V 9330 900 40  0000 C CNN
+F 1 "tbd" V 9257 901 40  0000 C CNN
 F 2 "~" V 9180 900 30  0000 C CNN
 F 3 "~" H 9250 900 30  0000 C CNN
@@
 P 7400 1900
 F 0 "Q?" H 7400 2090 60  0000 R CNN
-F 1 "MOSFET_P" H 7400 1720 60  0000 R CNN
+F 1 "DMP1045U" H 7400 1720 60  0000 R CNN
 F 2 "~" H 7400 1900 60  0000 C CNN
 F 3 "~" H 7400 1900 60  0000 C CNN
@@
 Connection ~ 6000 2800
 Wire Wire Line
-	4700 2000 4100 2000
+	3100 2000 4700 2000
 Wire Wire Line
 	4100 2000 4100 2100
+$Comp
+L TLV271 U?
+U 1 1 5532B295
+P 5350 5000
+F 0 "U?" H 5350 5000 60  0000 C CNN
+F 1 "TLV271" H 5350 4250 60  0000 C CNN
+F 2 "" H 5350 5000 60  0000 C CNN
+F 3 "" H 5350 5000 60  0000 C CNN
+	1    5350 5000
+	1    0    0    -1
+$EndComp
+Wire Wire Line
+	6800 3950 7900 3950
+Wire Wire Line
+	7900 3950 7900 6000
+Wire Wire Line
+	7900 6000 4600 6000
+Wire Wire Line
+	4600 6000 4600 5600
+Wire Wire Line
+	4600 5600 4750 5600
+$Comp
+L R R?
+U 1 1 5532B365
+P 6550 5600
+F 0 "R?" V 6630 5600 40  0000 C CNN
+F 1 "JUMPER" V 6557 5601 40  0000 C CNN
+F 2 "~" V 6480 5600 30  0000 C CNN
+F 3 "~" H 6550 5600 30  0000 C CNN
+	1    6550 5600
+	0    -1   -1   0
+$EndComp
+Wire Wire Line
+	5950 5600 6300 5600
+$Comp
+L R R?
+U 1 1 5532B4CB
+P 4350 5200
+F 0 "R?" V 4430 5200 40  0000 C CNN
+F 1 "JUMPER" V 4357 5201 40  0000 C CNN
+F 2 "~" V 4280 5200 30  0000 C CNN
+F 3 "~" H 4350 5200 30  0000 C CNN
+	1    4350 5200
+	0    -1   -1   0
+$EndComp
+Wire Wire Line
+	4600 5200 4750 5200
+Wire Wire Line
+	6800 5600 6800 4700
+Wire Wire Line
+	6800 4700 3900 4700
+Wire Wire Line
+	3900 4700 3900 5200
+Wire Wire Line
+	3600 5200 4100 5200
+$Comp
+L R R?
+U 1 1 5532B54B
+P 3350 5200
+F 0 "R?" V 3430 5200 40  0000 C CNN
+F 1 "tbd" V 3357 5201 40  0000 C CNN
+F 2 "~" V 3280 5200 30  0000 C CNN
+F 3 "~" H 3350 5200 30  0000 C CNN
+	1    3350 5200
+	0    -1   -1   0
+$EndComp
+Connection ~ 3900 5200
+$Comp
+L CSMALL C?
+U 1 1 5532B5A8
+P 2950 5400
+F 0 "C?" H 2975 5450 30  0000 L CNN
+F 1 "tbd" H 2975 5350 30  0000 L CNN
+F 2 "~" H 2950 5400 60  0000 C CNN
+F 3 "~" H 2950 5400 60  0000 C CNN
+	1    2950 5400
+	1    0    0    -1
+$EndComp
+Wire Wire Line
+	2500 5200 3100 5200
+Wire Wire Line
+	2950 5200 2950 5300
+Wire Wire Line
+	4750 5400 3800 5400
+Wire Wire Line
+	3800 5400 3800 6200
+Wire Wire Line
+	2500 5700 3800 5700
+Wire Wire Line
+	2950 5700 2950 5500
+$Comp
+L CSMALL C?
+U 1 1 5532B635
+P 6150 5350
+F 0 "C?" H 6175 5400 30  0000 L CNN
+F 1 "CSMALL" H 6175 5300 30  0000 L CNN
+F 2 "~" H 6150 5350 60  0000 C CNN
+F 3 "~" H 6150 5350 60  0000 C CNN
+	1    6150 5350
+	1    0    0    -1
+$EndComp
+Wire Wire Line
+	6150 5250 6150 5200
+Wire Wire Line
+	5950 5200 6400 5200
+Wire Wire Line
+	6150 5450 6150 6200
+Wire Wire Line
+	6150 6200 3800 6200
+Connection ~ 3800 5700
+$Comp
+L +3.3V #PWR?
+U 1 1 5532B6FE
+P 3100 1900
+F 0 "#PWR?" H 3100 1860 30  0001 C CNN
+F 1 "+3.3V" H 3100 2010 30  0000 C CNN
+F 2 "" H 3100 1900 60  0000 C CNN
+F 3 "" H 3100 1900 60  0000 C CNN
+	1    3100 1900
+	1    0    0    -1
+$EndComp
+Wire Wire Line
+	3100 2000 3100 1900
+Connection ~ 4100 2000
+$Comp
+L +3.3V #PWR?
+U 1 1 5532B74F
+P 6400 5100
+F 0 "#PWR?" H 6400 5060 30  0001 C CNN
+F 1 "+3.3V" H 6400 5210 30  0000 C CNN
+F 2 "" H 6400 5100 60  0000 C CNN
+F 3 "" H 6400 5100 60  0000 C CNN
+	1    6400 5100
+	1    0    0    -1
+$EndComp
+Wire Wire Line
+	6400 5200 6400 5100
+Connection ~ 6150 5200
+$Comp
+L POT RV?
+U 1 1 5532B7A2
+P 2500 5450
+F 0 "RV?" H 2500 5350 50  0000 C CNN
+F 1 "POT" H 2500 5450 50  0000 C CNN
+F 2 "~" H 2500 5450 60  0000 C CNN
+F 3 "~" H 2500 5450 60  0000 C CNN
+	1    2500 5450
+	0    -1   1    0
+$EndComp
+Connection ~ 2950 5200
+Connection ~ 2950 5700
+Text GLabel 1700 5450 0    60   Input ~ 0
+AUDIO OUT
+Wire Wire Line
+	2350 5450 1700 5450
 $EndSCHEMATC

Commit message: Schematics + License
Schematics support now ICSP connector.
Also the license file added.
Parts:
- added D?: DIODE, ~, symbol DIODE
- added P?: ICSP_CONN5, symbol CONN_5
- added P?: RESET_CONN_2, symbol CONN_2
- added R?: 4k7, ~, symbol R
Connections:
- wire segments 55 -> 79
Other:
- moved on the sheet: U?
Changed lines of the file:
@@
 L PIC18F14K50 U?
 U 1 1 5532862A
-P 5750 3750
-F 0 "U?" H 5650 3050 60  0000 C CNN
-F 1 "PIC18F14K50" H 5750 4350 60  0000 C CNN
-F 2 "~" H 5250 4300 60  0000 C CNN
-F 3 "~" H 5250 4300 60  0000 C CNN
-	1    5750 3750
+P 5750 3700
+F 0 "U?" H 5650 3000 60  0000 C CNN
+F 1 "PIC18F14K50" H 5750 4300 60  0000 C CNN
+F 2 "~" H 5250 4250 60  0000 C CNN
+F 3 "~" H 5250 4250 60  0000 C CNN
+	1    5750 3700
 	1    0    0    -1
 $EndComp
@@
 	1    0    0    -1
 $EndComp
-Wire Wire Line
-	7600 2000 8700 2000
-Wire Wire Line
-	8300 2000 8300 2200
-Wire Wire Line
-	8000 2200 8000 2000
-Connection ~ 8300 2000
 $Comp
 L GND #PWR?
@@
 	1    0    0    -1
 $EndComp
-Wire Wire Line
-	8300 2400 8300 2900
-Wire Wire Line
-	7800 2200 7600 2200
-Wire Wire Line
-	7600 2200 7600 2800
-Wire Wire Line
-	4100 2800 10300 2800
-Connection ~ 8300 2800
 $Comp
 L R R?
@@
 	0    -1   -1   0
 $EndComp
-Wire Wire Line
-	9850 1800 9850 1200
-Wire Wire Line
-	9850 1200 9500 1200
-Wire Wire Line
-	9000 1200 8400 1200
-Wire Wire Line
-	8400 1200 8400 1900
-Wire Wire Line
-	8400 1900 8700 1900
 $Comp
 L R R?
@@
 	0    -1   -1   0
 $EndComp
-Wire Wire Line
-	10100 900  9500 900
-Wire Wire Line
-	9000 900  8700 900
-Wire Wire Line
-	8700 900  8700 1800
-Wire Wire Line
-	10100 1300 10100 2000
-Wire Wire Line
-	9850 2000 10800 2000
 $Comp
 L CSMALL C?
@@
 	1    0    0    -1
 $EndComp
-Wire Wire Line
-	10300 700  10300 2200
-Connection ~ 10100 2000
-Wire Wire Line
-	10300 2800 10300 2400
 $Comp
 L +5V #PWR?
@@
 	1    0    0    -1
 $EndComp
-Wire Wire Line
-	10800 2000 10800 1900
-Connection ~ 10300 2000
 $Comp
 L MOSFET_P Q?
@@
 	0    1    1    0
 $EndComp
-Connection ~ 8000 2000
-Wire Wire Line
-	6800 700  10300 700
-Wire Wire Line
-	7400 700  7400 1700
 $Comp
 L DIODESCH D?
@@
 	0    1    1    0
 $EndComp
-Connection ~ 7400 700
-Wire Wire Line
-	6800 1100 6800 2000
-Wire Wire Line
-	5600 2000 7200 2000
 $Comp
 L CSMALL C?
@@
 	1    0    0    -1
 $EndComp
-Connection ~ 6800 2000
-Wire Wire Line
-	6200 2100 6200 2000
-Connection ~ 6200 2000
-Wire Wire Line
-	6200 2800 6200 2300
-Connection ~ 7600 2800
-Wire Wire Line
-	5600 2150 6000 2150
-Wire Wire Line
-	6000 2150 6000 2800
-Connection ~ 6200 2800
 $Comp
 L CP1 C?
@@
 	1    0    0    -1
 $EndComp
-Wire Wire Line
-	4100 2800 4100 2500
-Connection ~ 6000 2800
-Wire Wire Line
-	3100 2000 4700 2000
-Wire Wire Line
-	4100 2000 4100 2100
 $Comp
 L TLV271 U?
@@
 	1    0    0    -1
 $EndComp
-Wire Wire Line
-	6800 3950 7900 3950
-Wire Wire Line
-	7900 3950 7900 6000
-Wire Wire Line
-	7900 6000 4600 6000
-Wire Wire Line
-	4600 6000 4600 5600
-Wire Wire Line
-	4600 5600 4750 5600
 $Comp
 L R R?
@@
 	0    -1   -1   0
 $EndComp
-Wire Wire Line
-	5950 5600 6300 5600
 $Comp
 L R R?
@@
 	0    -1   -1   0
 $EndComp
-Wire Wire Line
-	4600 5200 4750 5200
-Wire Wire Line
-	6800 5600 6800 4700
-Wire Wire Line
-	6800 4700 3900 4700
-Wire Wire Line
-	3900 4700 3900 5200
-Wire Wire Line
-	3600 5200 4100 5200
 $Comp
 L R R?
@@
 	0    -1   -1   0
 $EndComp
-Connection ~ 3900 5200
 $Comp
 L CSMALL C?
@@
 	1    0    0    -1
 $EndComp
-Wire Wire Line
-	2500 5200 3100 5200
-Wire Wire Line
-	2950 5200 2950 5300
-Wire Wire Line
-	4750 5400 3800 5400
-Wire Wire Line
-	3800 5400 3800 6200
-Wire Wire Line
-	2500 5700 3800 5700
-Wire Wire Line
-	2950 5700 2950 5500
 $Comp
 L CSMALL C?
@@
 	1    0    0    -1
 $EndComp
-Wire Wire Line
-	6150 5250 6150 5200
-Wire Wire Line
-	5950 5200 6400 5200
-Wire Wire Line
-	6150 5450 6150 6200
-Wire Wire Line
-	6150 6200 3800 6200
-Connection ~ 3800 5700
 $Comp
 L +3.3V #PWR?
@@
 	1    0    0    -1
 $EndComp
-Wire Wire Line
-	3100 2000 3100 1900
-Connection ~ 4100 2000
 $Comp
 L +3.3V #PWR?
@@
 	1    0    0    -1
 $EndComp
-Wire Wire Line
-	6400 5200 6400 5100
-Connection ~ 6150 5200
 $Comp
 L POT RV?
@@
 	0    -1   1    0
 $EndComp
+Text GLabel 1700 5450 0    60   Input ~ 0
+AUDIO OUT
+$Comp
+L CONN_5 P?
+U 1 1 5532BCAA
+P 10300 3400
+F 0 "P?" V 10250 3400 50  0000 C CNN
+F 1 "ICSP_CONN5" V 10350 3400 50  0000 C CNN
+F 2 "" H 10300 3400 60  0000 C CNN
+F 3 "" H 10300 3400 60  0000 C CNN
+	1    10300 3400
+	1    0    0    -1
+$EndComp
+$Comp
+L R R?
+U 1 1 5532BDB1
+P 3500 3150
+F 0 "R?" V 3580 3150 40  0000 C CNN
+F 1 "4k7" V 3507 3151 40  0000 C CNN
+F 2 "~" V 3430 3150 30  0000 C CNN
+F 3 "~" H 3500 3150 30  0000 C CNN
+	1    3500 3150
+	1    0    0    -1
+$EndComp
+$Comp
+L DIODE D?
+U 1 1 5532BDC0
+P 3800 3600
+F 0 "D?" H 3800 3700 40  0000 C CNN
+F 1 "DIODE" H 3800 3500 40  0000 C CNN
+F 2 "~" H 3800 3600 60  0000 C CNN
+F 3 "~" H 3800 3600 60  0000 C CNN
+	1    3800 3600
+	1    0    0    -1
+$EndComp
+$Comp
+L CONN_2 P?
+U 1 1 5532BEA6
+P 3100 3150
+F 0 "P?" V 3050 3150 40  0000 C CNN
+F 1 "RESET_CONN_2" V 3150 3150 40  0000 C CNN
+F 2 "" H 3100 3150 60  0000 C CNN
+F 3 "" H 3100 3150 60  0000 C CNN
+	1    3100 3150
+	0    -1   -1   0
+$EndComp
+Wire Wire Line
+	7600 2000 8700 2000
+Wire Wire Line
+	8300 2000 8300 2200
+Wire Wire Line
+	8000 2200 8000 2000
+Connection ~ 8300 2000
+Wire Wire Line
+	8300 2400 8300 2900
+Wire Wire Line
+	7800 2200 7600 2200
+Wire Wire Line
+	7600 2200 7600 2800
+Wire Wire Line
+	2700 2800 10300 2800
+Connection ~ 8300 2800
+Wire Wire Line
+	9850 1800 9850 1200
+Wire Wire Line
+	9850 1200 9500 1200
+Wire Wire Line
+	9000 1200 8400 1200
+Wire Wire Line
+	8400 1200 8400 1900
+Wire Wire Line
+	8400 1900 8700 1900
+Wire Wire Line
+	10100 900  9500 900
+Wire Wire Line
+	9000 900  8700 900
+Wire Wire Line
+	8700 900  8700 1800
+Wire Wire Line
+	10100 1300 10100 2000
+Wire Wire Line
+	9850 2000 10800 2000
+Wire Wire Line
+	10300 700  10300 2200
+Connection ~ 10100 2000
+Wire Wire Line
+	10300 2800 10300 2400
+Wire Wire Line
+	10800 2000 10800 1900
+Connection ~ 10300 2000
+Connection ~ 8000 2000
+Wire Wire Line
+	6800 700  10300 700
+Wire Wire Line
+	7400 700  7400 1700
+Connection ~ 7400 700
+Wire Wire Line
+	6800 2000 6800 1100
+Wire Wire Line
+	5600 2000 7200 2000
+Connection ~ 6800 2000
+Wire Wire Line
+	6200 2100 6200 2000
+Connection ~ 6200 2000
+Wire Wire Line
+	6200 2800 6200 2300
+Connection ~ 7600 2800
+Wire Wire Line
+	5600 2150 6000 2150
+Wire Wire Line
+	6000 2150 6000 2800
+Connection ~ 6200 2800
+Wire Wire Line
+	4100 2800 4100 2500
+Connection ~ 6000 2800
+Wire Wire Line
+	3100 2000 4700 2000
+Wire Wire Line
+	4100 2000 4100 2100
+Wire Wire Line
+	6800 3900 7900 3900
+Wire Wire Line
+	7900 3900 7900 6000
+Wire Wire Line
+	7900 6000 4600 6000
+Wire Wire Line
+	4600 6000 4600 5600
+Wire Wire Line
+	4600 5600 4750 5600
+Wire Wire Line
+	5950 5600 6300 5600
+Wire Wire Line
+	4600 5200 4750 5200
+Wire Wire Line
+	6800 5600 6800 4700
+Wire Wire Line
+	6800 4700 3900 4700
+Wire Wire Line
+	3900 4700 3900 5200
+Wire Wire Line
+	3600 5200 4100 5200
+Connection ~ 3900 5200
+Wire Wire Line
+	2500 5200 3100 5200
+Wire Wire Line
+	2950 5200 2950 5300
+Wire Wire Line
+	4750 5400 3800 5400
+Wire Wire Line
+	3800 5400 3800 6200
+Wire Wire Line
+	2500 5700 3800 5700
+Wire Wire Line
+	2950 5700 2950 5500
+Wire Wire Line
+	6150 5250 6150 5200
+Wire Wire Line
+	5950 5200 6400 5200
+Wire Wire Line
+	6150 5450 6150 6200
+Wire Wire Line
+	6150 6200 3800 6200
+Connection ~ 3800 5700
+Wire Wire Line
+	3100 2000 3100 1900
+Connection ~ 4100 2000
+Wire Wire Line
+	6400 5200 6400 5100
+Connection ~ 6150 5200
 Connection ~ 2950 5200
 Connection ~ 2950 5700
-Text GLabel 1700 5450 0    60   Input ~ 0
-AUDIO OUT
 Wire Wire Line
 	2350 5450 1700 5450
+Wire Wire Line
+	4000 3600 4700 3600
+Wire Wire Line
+	4200 2900 4200 3750
+Wire Wire Line
+	4200 2900 7800 2900
+Wire Wire Line
+	7800 2900 7800 3200
+Wire Wire Line
+	7800 3200 9900 3200
+Connection ~ 4200 3600
+Wire Wire Line
+	3500 3600 3500 3400
+Wire Wire Line
+	3200 3500 3200 3750
+Wire Wire Line
+	3000 3500 3000 3600
+Wire Wire Line
+	3000 3600 2700 3600
+Wire Wire Line
+	2700 3600 2700 2800
+Connection ~ 4100 2800
+Wire Wire Line
+	3500 2900 3500 2000
+Connection ~ 3500 2000
+Wire Wire Line
+	3500 3600 3600 3600
+Wire Wire Line
+	3200 3750 4200 3750
+$Comp
+L +3.3V #PWR?
+U 1 1 5532C128
+P 9700 4200
+F 0 "#PWR?" H 9700 4160 30  0001 C CNN
+F 1 "+3.3V" H 9700 4310 30  0000 C CNN
+F 2 "" H 9700 4200 60  0000 C CNN
+F 3 "" H 9700 4200 60  0000 C CNN
+	1    9700 4200
+	1    0    0    -1
+$EndComp
+Wire Wire Line
+	9700 4200 9400 4200
+Wire Wire Line
+	9400 4200 9400 3300
+Wire Wire Line
+	9400 3300 9900 3300
+Wire Wire Line
+	9900 3400 9500 3400
+Wire Wire Line
+	9500 3400 9500 2800
+Connection ~ 9500 2800
+Wire Wire Line
+	9900 3500 7450 3500
+Wire Wire Line
+	7450 3500 7450 3400
+Wire Wire Line
+	7450 3400 6800 3400
+Wire Wire Line
+	9900 3600 7350 3600
+Wire Wire Line
+	7350 3600 7350 3500
+Wire Wire Line
+	7350 3500 6800 3500
 $EndSCHEMATC

Commit message: More work on schematics
Now supporting PIC oscillator, jumper line for UART TX and audio
in/carrier detect.
Parts:
- added C? (x2): tbd, ~, symbol CSMALL
- added C?: 0uF1, ~, symbol CSMALL
- added P?: UART_TX_JUMPER, symbol CONN_2
- added RV?: 10k, ~, symbol POT
- added X?: 10MHz, ~, symbol CRYSTAL
- RV?: value POT -> 10k
Connections:
- net labels added: AUDIO IN, UART_TX
- wire segments 79 -> 104
Other:
- moved on the sheet: R?, RV?, U?

Commit message: Schematics mostly done
Schematics are only lacking 2 LEDs and all the buttons and a switch.
Also need to revisit the USB connection.
Parts:
- added J?: USB_MINI, ~, symbol USB_MINI
- added P?: I2C_SCREEN, symbol CONN_4
- added R? (x2): JUMPWIRE, ~, symbol R
Connections:
- net labels added: UART_RX
- wire segments 104 -> 131
Changed lines of the file:
@@
 LIBS:valves
 LIBS:remote_bt_shutter-cache
+LIBS:imx23_phone-cache
 LIBS:korsotracker-cache
 EELAYER 27 0
@@
 $EndComp
 $Comp
-L +3.3V #PWR?
-U 1 1 5532C128
-P 9700 4200
-F 0 "#PWR?" H 9700 4160 30  0001 C CNN
-F 1 "+3.3V" H 9700 4310 30  0000 C CNN
-F 2 "" H 9700 4200 60  0000 C CNN
-F 3 "" H 9700 4200 60  0000 C CNN
-	1    9700 4200
-	1    0    0    -1
-$EndComp
-$Comp
 L CRYSTAL X?
 U 1 1 5532C410
@@
 	9400 3300 9900 3300
 Wire Wire Line
-	9400 4200 9400 3300
-Wire Wire Line
-	9700 4200 9400 4200
-Wire Wire Line
 	4200 3750 3200 3750
 Wire Wire Line
@@
 	4600 7050 4600 6650
 Wire Wire Line
-	7900 7050 4600 7050
-Wire Wire Line
-	7900 3900 7900 7050
-Wire Wire Line
-	6800 3900 7900 3900
+	7000 7050 4600 7050
+Wire Wire Line
+	7000 3900 7000 7050
+Wire Wire Line
+	6800 3900 7000 3900
 Wire Wire Line
 	4100 2000 4100 2100
@@
 Connection ~ 8300 2800
 Wire Wire Line
-	1400 2800 10300 2800
+	1400 2800 11000 2800
 Wire Wire Line
 	7600 2200 7600 2800
@@
 Text GLabel 1200 4200 0    60   Output ~ 0
 UART_TX
-Wire Wire Line
-	2500 4200 1200 4200
 $Comp
 L POT RV?
@@
 Wire Wire Line
 	1600 5850 1600 5950
+$Comp
+L R R?
+U 1 1 5532DD5A
+P 1650 4200
+F 0 "R?" V 1730 4200 40  0000 C CNN
+F 1 "JUMPWIRE" V 1657 4201 40  0000 C CNN
+F 2 "~" V 1580 4200 30  0000 C CNN
+F 3 "~" H 1650 4200 30  0000 C CNN
+	1    1650 4200
+	0    -1   -1   0
+$EndComp
+$Comp
+L R R?
+U 1 1 5532DD6D
+P 1650 4600
+F 0 "R?" V 1730 4600 40  0000 C CNN
+F 1 "JUMPWIRE" V 1657 4601 40  0000 C CNN
+F 2 "~" V 1580 4600 30  0000 C CNN
+F 3 "~" H 1650 4600 30  0000 C CNN
+	1    1650 4600
+	0    -1   -1   0
+$EndComp
+Text GLabel 1200 4600 0    60   Input ~ 0
+UART_RX
+Wire Wire Line
+	1400 4200 1200 4200
+Wire Wire Line
+	1900 4200 2500 4200
+Wire Wire Line
+	1400 4600 1200 4600
+Wire Wire Line
+	6800 4100 6900 4100
+Wire Wire Line
+	6900 4100 6900 4600
+Wire Wire Line
+	6900 4600 3000 4600
+Wire Wire Line
+	3000 4600 3000 4700
+Wire Wire Line
+	3000 4700 1950 4700
+Wire Wire Line
+	1950 4700 1950 4600
+Wire Wire Line
+	1950 4600 1900 4600
+$Comp
+L CONN_4 P?
+U 1 1 5532E038
+P 10300 4000
+F 0 "P?" V 10250 4000 50  0000 C CNN
+F 1 "I2C_SCREEN" V 10350 4000 50  0000 C CNN
+F 2 "" H 10300 4000 60  0000 C CNN
+F 3 "" H 10300 4000 60  0000 C CNN
+	1    10300 4000
+	1    0    0    -1
+$EndComp
+$Comp
+L +3.3V #PWR?
+U 1 1 5532C128
+P 10800 3000
+F 0 "#PWR?" H 10800 2960 30  0001 C CNN
+F 1 "+3.3V" H 10800 3110 30  0000 C CNN
+F 2 "" H 10800 3000 60  0000 C CNN
+F 3 "" H 10800 3000 60  0000 C CNN
+	1    10800 3000
+	1    0    0    -1
+$EndComp
+Wire Wire Line
+	9400 3300 9400 3000
+Wire Wire Line
+	9200 3000 10800 3000
+Wire Wire Line
+	9950 3850 9200 3850
+Wire Wire Line
+	9200 3850 9200 3000
+Connection ~ 9400 3000
+Wire Wire Line
+	9950 3950 9100 3950
+Wire Wire Line
+	9100 3950 9100 2800
+Connection ~ 9100 2800
+Wire Wire Line
+	6800 4200 9400 4200
+Wire Wire Line
+	9400 4200 9400 4050
+Wire Wire Line
+	9400 4050 9950 4050
+Wire Wire Line
+	6800 4000 9300 4000
+Wire Wire Line
+	9300 4000 9300 4150
+Wire Wire Line
+	9300 4150 9950 4150
+$Comp
+L USB_MINI J?
+U 1 1 5532E5CD
+P 9800 4400
+F 0 "J?" H 9800 4400 60  0000 C CNN
+F 1 "USB_MINI" H 9800 4400 60  0000 C CNN
+F 2 "~" H 9800 4400 60  0000 C CNN
+F 3 "~" H 9800 4400 60  0000 C CNN
+	1    9800 4400
+	-1   0    0    -1
+$EndComp
+Wire Wire Line
+	9200 4650 9000 4650
+Wire Wire Line
+	9000 4650 9000 3600
+Connection ~ 9000 3600
+Wire Wire Line
+	9200 4750 8900 4750
+Wire Wire Line
+	8900 4750 8900 3500
+Connection ~ 8900 3500
+Wire Wire Line
+	10400 4650 10600 4650
+Wire Wire Line
+	10600 4650 10600 3000
+Connection ~ 10600 3000
+Wire Wire Line
+	10400 4750 11000 4750
+Wire Wire Line
+	11000 4750 11000 2800
+Connection ~ 10300 2800
 $EndSCHEMATC
