File: hardware/yaatracker/yaatracker.sch (KiCad schematic (older format))
At the start: 34 parts

Commit message: Schematics before check
Schematics are ready to be checked.
Parts:
- added C? (x3): CSMALL, ~, symbol CSMALL
- added D? (x2): LED, ~, symbol LED
- added P?: GPIO10_GND_JUMPER, symbol CONN_2
- added P?: MBUTTON3, symbol CONN_2
- added P?: MBUTTON2, symbol CONN_2
- added P?: MBUTTON1, symbol CONN_2
- added R? (x2): 60, ~, symbol R
- added R? (x3): 1k, ~, symbol R
- added R? (x2): tbd, ~, symbol R
- added R? (x3): R, ~, symbol R
- added T?: BSV52, ~, symbol BSV52
Connections:
- net labels added: PTT
- wire segments 131 -> 248
- no-connect marks 0 -> 2
Other:
- moved on the sheet: D?, P?, R?, X?

Commit message: Schematics work
Working to get a good pcb
Parts:
- C?: value CSMALL -> tbd
- C?: value CSMALL -> 270nF
- C?: value CSMALL -> 0uF1
- R?: value R -> tbd
- R?: value R -> 1k
- R?: value R -> 47k
Connections:
- no-connect marks 2 -> 3
Changed lines of the file:
@@
 P 6150 6400
 F 0 "C?" H 6175 6450 30  0000 L CNN
-F 1 "CSMALL" H 6175 6350 30  0000 L CNN
+F 1 "tbd" H 6175 6350 30  0000 L CNN
 F 2 "~" H 6150 6400 60  0000 C CNN
 F 3 "~" H 6150 6400 60  0000 C CNN
@@
 P 7000 3200
 F 0 "C?" H 7025 3250 30  0000 L CNN
-F 1 "CSMALL" H 7025 3150 30  0000 L CNN
+F 1 "270nF" H 7025 3150 30  0000 L CNN
 F 2 "~" H 7000 3200 60  0000 C CNN
 F 3 "~" H 7000 3200 60  0000 C CNN
@@
 P 4300 4550
 F 0 "R?" V 4380 4550 40  0000 C CNN
-F 1 "R" V 4307 4551 40  0000 C CNN
+F 1 "tbd" V 4307 4551 40  0000 C CNN
 F 2 "~" V 4230 4550 30  0000 C CNN
 F 3 "~" H 4300 4550 30  0000 C CNN
@@
 P 4050 5600
 F 0 "R?" V 4130 5600 40  0000 C CNN
-F 1 "R" V 4057 5601 40  0000 C CNN
+F 1 "1k" V 4057 5601 40  0000 C CNN
 F 2 "~" V 3980 5600 30  0000 C CNN
 F 3 "~" H 4050 5600 30  0000 C CNN
@@
 P 4800 5150
 F 0 "R?" V 4880 5150 40  0000 C CNN
-F 1 "R" V 4807 5151 40  0000 C CNN
+F 1 "47k" V 4807 5151 40  0000 C CNN
 F 2 "~" V 4730 5150 30  0000 C CNN
 F 3 "~" H 4800 5150 30  0000 C CNN
@@
 P 5200 5350
 F 0 "C?" H 5225 5400 30  0000 L CNN
-F 1 "CSMALL" H 5225 5300 30  0000 L CNN
+F 1 "0uF1" H 5225 5300 30  0000 L CNN
 F 2 "~" H 5200 5350 60  0000 C CNN
 F 3 "~" H 5200 5350 60  0000 C CNN
@@
 	5200 5450 5200 5850
 Connection ~ 5200 5850
+NoConn ~ 4700 2150
 $EndSCHEMATC

Commit message: SCHEMATICS DONE
Schematics should be now ready.
Parts:
- removed R? (x2): JUMPWIRE, ~, symbol R
- added P?: TP_URX, ~, symbol TST
- added P?: TP_UTX, ~, symbol TST
- added P?: TP_TON1, ~, symbol TST
- added P?: TON2, ~, symbol TST
- added P?: GPS_DE9, symbol CONN_4
- added P?: RADIO_DE9, symbol CONN_5
- added P?: R_VCC, symbol CONN_2
- added R? (x2): 4k7, ~, symbol R
- added R?: 100K, ~, symbol R
- C? (x2): value tbd -> 15pF
- P?: value LIPO -> BATT
Connections:
- net labels added: 3V3, AUDIO_IN, AUDIO_OUT, R_VOUT
- net labels removed: +5V
- wire segments 248 -> 232
Other:
- moved on the sheet: D?, R?

Commit message: Schematics after ERC
Some fixes after ERC. ERC still complains but only warnings - nothing
serious that would need to be fixed for now.
Parts:
- gave numbers to parts that had none: 62
Connections:
- net labels removed: AUDIO IN, AUDIO OUT
- wire segments 232 -> 216

Commit message: PCB layout power circuit
Started the power circuit layout of the PCB.
Connections:
- wire segments 216 -> 217
Changed lines of the file:
@@
 Sheet 1 1
 Title "YAAT, an APRS Tracker"
-Date "20 apr 2015"
+Date "24 apr 2015"
 Rev ""
 Comp ""
@@
 Wire Wire Line
 	800  2800 10600 2800
+Wire Wire Line
+	8600 2800 8600 1900
+Connection ~ 8600 1900
+Connection ~ 8600 2800
 $EndSCHEMATC
