File: hardware/yaatracker/yaatracker.sch (KiCad schematic (older format))
At the start: 62 parts, among them J1 USB_MINI, P1 TP_URX, P10 BATT, P11 MBUTTON2, P12 ICSP_CONN5, P13 I2C_SCREEN, P14 R_VCC, P15 GPS_DE9, P16 RADIO_DE9, P2 GPIO10_GND_JUMPER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

Commit message: PCB layout last switch
Added and routed another switch successfully.
Parts:
- added P17: SW5, symbol CONN_2
Connections:
- wire segments 218 -> 222
