File: hardware/yaatracker/yaatracker.kicad_pcb (KiCad board)
At the start: 2 copper layers, 47.6 x 49.4 mm, 68 parts, among them J1 USB_MINI, P1 TP_URX, P10 BATT, P11 MBUTTON2, P12 ICSP_CONN5, P13 I2C_SCREEN, P14 R_VCC, P15 GPS_DE9, P16 RADIO_DE9, P17 SW5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

Commit message: PCB version 1.0
PCB done, ready for printing. PCB version 1.0.
Other:
- board text added: "Karri Kivelä 04/2015, karrister@gmail.com"
- board text added: "YAAT, an APRS tracker Karri Kivelä 04/2015"
- board text added: "www.karrikivela.fi"
Changed lines of the file:
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@@
     (links 121)
     (no_connects 0)
-    (area 0 0 0 0)
+    (area 104.679045 117.949999 153.050001 167.461401)
     (thickness 1.6)
-    (drawings 4)
+    (drawings 8)
     (tracks 574)
     (zones 0)
@@
     (visible_elements 7FFFFFFF)
     (pcbplotparams
-      (layerselection 3178497)
+      (layerselection 284196865)
       (usegerberextensions true)
       (excludeedgelayer true)
@@
       (outputformat 1)
       (mirror false)
-      (drillshape 1)
+      (drillshape 0)
       (scaleselection 1)
       (outputdirectory ""))
@@
     )
   )
+  (gr_text "YAAT, an APRS tracker\nKarri Kivelä 04/2015" (at 151.4348 136.398 270) (layer F.SilkS)
+    (effects (font (size 1.3 1.3) (thickness 0.3)))
+  )
+  (gr_text www.karrikivela.fi (at 145.0594 166.4716) (layer F.SilkS)
+    (effects (font (size 1.1 1.1) (thickness 0.275)))
+  )
+  (gr_text www.karrikivela.fi (at 142.0495 166.5224) (layer B.SilkS)
+    (effects (font (size 1.1 1.1) (thickness 0.275)) (justify mirror))
+  )
+  (gr_text "Karri Kivelä 04/2015, karrister@gmail.com" (at 151.3967 141.1732 270) (layer B.SilkS)
+    (effects (font (size 1.2 1.2) (thickness 0.3)) (justify mirror))
+  )
   (gr_line (start 153 118) (end 105.3846 118) (angle 90) (layer Edge.Cuts) (width 0.1))
